File: hw/driver.kicad_sch (KiCad schematic)
At the start: 9 parts, among them U3 DRV8353S

Commit message: Route the 6-layer board and finalize parts for ordering
The 45 x 45 mm board is fully routed on six layers (F / GND / SIG /
SIG / PWR / B, 2 oz outer, 1 oz inner): DRC 0 errors, 0 unconnected,
schematic parity 0. Four layers could not route the DRV-to-MCU links
without moving the power or input stage.

- Encoder shares the DRV8353's SPI3 bus, as on the PoC; PA5-PA7 are
  unused. R25 pulls DRV nSCS up, since the DRV's logic inputs have an
  internal pull-down. The SDO / MISO pin-type warning is an ERC
  exclusion with a note.
- MCU is now the STM32G473CEU6: the G474 without the unused HRTIM,
  checked pin for pin against both datasheets, in stock and cheaper.
- Male XT30PW-M power connectors, HCS1206 shunts, SWD pads at the
  board edge.
- Design doc and review notes updated for the new stack-up, shared
  bus and MCU.

Co-Authored-By: Claude Opus 5.5 <noreply@anthropic.com>
Parts:
- added R25: 10k 1%, Resistor_SMD:R_0402_1005Metric, symbol Device:R
Connections:
- net +3V3: now also R25.1
- net DRV_nSCS: now also R25.2
Other:
- note added: "DRV8353S external parts (SLVSDY6A Table 21, Fig. 63): C18 VM 0.1 uF VM-rated (bulk on Power sheet provides >= 10 uF) C19 VCP to VDRAIN 1 uF 16 V+ C20 CPH-CPL 47 nF VDRAIN-rated C21 VGLS 1 uF 16 V+ C22 DVDD 1 uF 6.3 V+ C23 VREF 0.1 uF R6 nFAULT 10k, R7 SDO 1k pull-ups to 3.3 V (open drain, Fig. 63). Internal: nSCS 50k pull-up to DVDD (5 V): MCU pin must be FT (PA15). ENABLE, INHx/INLx, SCLK, SDI h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"
- note removed: "DRV8353S external parts (SLVSDY6A Table 21, Fig. 63): C18 VM 0.1 uF VM-rated (bulk on Power sheet provides >= 10 uF) C19 VCP to VDRAIN 1 uF 16 V+ C20 CPH-CPL 47 nF VDRAIN-rated C21 VGLS 1 uF 16 V+ C22 DVDD 1 uF 6.3 V+ C23 VREF 0.1 uF R6 nFAULT 10k, R7 SDO 1k pull-ups to 3.3 V (open drain, Fig. 63). Internal: nSCS 50k pull-up to DVDD (5 V): MCU pin must be FT (PB7). ENABLE, INHx/INLx, SCLK, SDI ha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"
Changed lines of the file:
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@@
 		(comment 2 "specs/pmsm-controller/design-electronics.md")
 	)
-	(text "DRV8353S external parts (SLVSDY6A Table 21, Fig. 63):\nC18 VM 0.1 uF VM-rated (bulk on Power sheet provides >= 10 uF)\nC19 VCP to VDRAIN 1 uF 16 V+     C20 CPH-CPL 47 nF VDRAIN-rated\nC21 VGLS 1 uF 16 V+     C22 DVDD 1 uF 6.3 V+     C23 VREF 0.1 uF\nR6 nFAULT 10k, R7 SDO 1k pull-ups to 3.3 V (open drain, Fig. 63).\nInternal: nSCS 50k pull-up to DVDD (5 V): MCU pin must be FT (PB7).\nENABLE, INHx/INLx, SCLK, SDI have 100k pull-downs: bridge off in MCU reset.\nVDRAIN: route to the high-side MOSFET drains. VREF = MCU 3.3 V (ratiometric ADC).\nIdle = all INHx/INLx low (ENABLE low = sleep, registers reset)."
+	(text "DRV8353S external parts (SLVSDY6A Table 21, Fig. 63):\nC18 VM 0.1 uF VM-rated (bulk on Power sheet provides >= 10 uF)\nC19 VCP to VDRAIN 1 uF 16 V+     C20 CPH-CPL 47 nF VDRAIN-rated\nC21 VGLS 1 uF 16 V+     C22 DVDD 1 uF 6.3 V+     C23 VREF 0.1 uF\nR6 nFAULT 10k, R7 SDO 1k pull-ups to 3.3 V (open drain, Fig. 63).\nInternal: nSCS 50k pull-up to DVDD (5 V): MCU pin must be FT (PA15).\nENABLE, INHx/INLx, SCLK, SDI have 100k pull-downs: bridge off in MCU reset.\nVDRAIN: route to the high-side MOSFET drains. VREF = MCU 3.3 V (ratiometric ADC).\nIdle = all INHx/INLx low (ENABLE low = sleep, registers reset)."
 		(exclude_from_sim no)
 		(at 22.86 236.22 0)
@@
 					(unit 1)
 				)
+			)
+		)
+	)
+	(wire
+		(pts
+			(xy 139.7 196.85) (xy 139.7 194.31)
+		)
+		(stroke
+			(width 0)
+			(type default)
+		)
+	)
+	(wire
+		(pts
+			(xy 139.7 204.47) (xy 139.7 207.01)
+		)
+		(stroke
+			(width 0)
+			(type default)
+		)
+	)
+	(hierarchical_label "DRV_nSCS"
+		(shape output)
+		(at 139.7 207.01 270)
+		(effects
+			(font
+				(size 1.27 1.27)
+			)
+			(justify right)
+		)
+	)
+	(symbol
+		(lib_id "power:+3V3")
+		(at 139.7 194.31 0)
+		(unit 1)
+		(body_style 1)
+		(exclude_from_sim no)
+		(in_bom yes)
+		(on_board yes)
+		(in_pos_files yes)
+		(dnp no)
+		(property "Reference" "#PWRDRI13"
+			(at 139.7 190.5 0)
+			(hide yes)
+			(show_name no)
+			(do_not_autoplace no)
+			(effects
+				(font
+					(size 1.27 1.27)
+				)
+				(justify left)
+			)
+		)
+		(property "Value" "+3V3"
+			(at 139.7 189.23 0)
+			(show_name no)
+			(do_not_autoplace no)
+			(effects
+				(font
+					(size 1.27 1.27)
+				)
+			)
+		)
+		(property "Footprint" ""
+			(at 139.7 194.31 0)
+			(show_name no)
+			(do_not_autoplace no)
+			(effects
+				(font
+					(size 1.27 1.27)
+				)
+			)
+		)
+		(property "Datasheet" ""
+			(at 139.7 194.31 0)
+			(show_name no)
+			(do_not_autoplace no)
+			(effects
+				(font
+					(size 1.27 1.27)
+				)
+			)
+		)
+		(property "Description" ""
+			(at 139.7 194.31 0)
+			(show_name no)
+			(do_not_autoplace no)
+			(effects
+				(font
+					(size 1.27 1.27)
+				)
+			)
+		)
+		(pin "1"
+		)
+		(instances
+			(project "foc_controller"
+				(path "/dc3b1c6f-161a-46e4-9985-32c8fd205458/114a6df9-ba32-495c-a887-4cc1990c8360"
+					(reference "#PWRDRI13")
+					(unit 1)
+				)
+			)
+		)
+	)
+	(symbol
+		(lib_id "Device:R")
+		(at 139.7 200.66 0)
+		(unit 1)
+		(body_style 1)
+		(exclude_from_sim no)
+		(in_bom yes)
+		(on_board yes)
+		(in_pos_files yes)
+		(dnp no)
+		(property "Reference" "R25"
+			(at 142.24 199.39 0)
+			(show_name no)
+			(do_not_autoplace no)
+			(effects
+				(font
+					(size 1.27 1.27)
+				)
+				(justify left)
+			)
+		)
+		(property "Value" "10k 1%"
+			(at 142.24 201.93 0)
+			(show_name no)
+			(do_not_autoplace no)
+			(effects
+				(font
+					(size 1.27 1.27)
+				)
+				(justify left)
+			)
+		)
+		(property "Footprint" "Resistor_SMD:R_0402_1005Metric"
+			(at 137.922 200.66 90)
+			(hide yes)
+			(show_name no)
+			(do_not_autoplace no)
+			(effects
+				(font
+					(size 1.27 1.27)
+				)
+			)
+		)
+		(property "Datasheet" ""
+			(at 139.7 200.66 0)
+			(show_name no)
+			(do_not_autoplace no)
+			(effects
+				(font
+					(size 1.27 1.27)
+				)
+			)
+		)
+		(property "Description" ""
+			(at 139.7 200.66 0)
+			(show_name no)
+			(do_not_autoplace no)
+			(effects
+				(font
+					(size 1.27 1.27)
+				)
+			)
+		)
+		(property "LCSC" "C25744"
+			(at 142.24 205.7399 0)
+			(hide yes)
+			(show_name no)
+			(do_not_autoplace no)
+			(effects
+				(font
+					(size 1.27 1.27)
+				)
+				(justify left)
+			)
+		)
+		(property "MPN" "0402WGF1002TCE"
+			(at 142.24 205.7399 0)
+			(hide yes)
+			(show_name no)
+			(do_not_autoplace no)
+			(effects
+				(font
+					(size 1.27 1.27)
+				)
+				(justify left)
+			)
+		)
+		(pin "1"
+		)
+		(pin "2"
+		)
+		(instances
+			(project "foc_controller"
+				(path "/dc3b1c6f-161a-46e4-9985-32c8fd205458/114a6df9-ba32-495c-a887-4cc1990c8360"
+					(reference "R25")
+					(unit 1)
+				)
