File: hw/encoder.kicad_sch (KiCad schematic)
At the start: 2 parts, among them U5 AS5047P

Commit message: Apply schematic review fixes and connector changes
- Remove the RC snubber pads (ringing handled by layout and IDRIVE)
  and renumber R/C references to close the gap.
- CAN connectors: JST-GH 3-pin (CANH, CANL, GND).
- Power connectors: XT30PW-F female for both bus IN and OUT so the
  live side of every link is shrouded; polarity checked on a real
  part (pad 1 GND under the rounded end, pad 2 VBUS under the flat
  end). Male XT30 footprint, model and datasheet removed.
- AS5047P CSn 10k pull-up so encoder inputs never float while the
  MCU is in reset or ROM DFU.
- LM5008A RT 180k -> 240k: on-time stays >= 400 ns at 54 V across
  the TON spread.
- Every BOM line checked in stock against JLCPCB's assembly library.
- Kelvin-tap placement added to the layout rules.

Co-Authored-By: Claude Opus 5.5 <noreply@anthropic.com>
Parts:
- added R24: 10k 1%, Resistor_SMD:R_0402_1005Metric, symbol Device:R
Connections:
- net +3V3: now also R24.1
- net ENC_CS: now also R24.2
Other:
- note added: "AS5047P 3.3 V operation: VDD and VDD3V3 tied to 3.3 V, one 100 nF (DS000324 Fig. 10). TEST (pin 5) to GND per pin table. ABI / UVW / PWM outputs unused. R24 holds CSn high while the MCU is in reset or ROM DFU (inputs must not float, DS p.4). SPI mode 1, up to 10 MHz, on its own SPI port (SPI3). Place alone on the motor-facing side at the board center. Magnet 6 x 2.5 mm diametric, gap 1 to 2 mm. K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"
- note removed: "AS5047P 3.3 V operation: VDD and VDD3V3 tied to 3.3 V, one 100 nF (DS000324 Fig. 10). TEST (pin 5) to GND per pin table. ABI / UVW / PWM outputs unused. SPI mode 1, up to 10 MHz, on its own SPI port (SPI3). Place alone on the motor-facing side at the board center. Magnet 6 x 2.5 mm diametric, gap 1 to 2 mm. Keep phase and pass-through currents >= 12 mm away."
Changed lines of the file:
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@@
 		(instances
 			(project "encoder"
-				(path "/23e15ccf-2162-4caa-a05b-71e788486361/627dfe32-6c71-41ac-99ad-61f4ee65e4fe"
+				(path "/dc3b1c6f-161a-46e4-9985-32c8fd205458/9673b332-b1ed-481c-ad2c-77a34f76cbb1"
 					(reference "U5")
 					(unit 1)
@@
 		(instances
 			(project "encoder"
-				(path "/23e15ccf-2162-4caa-a05b-71e788486361/627dfe32-6c71-41ac-99ad-61f4ee65e4fe"
+				(path "/dc3b1c6f-161a-46e4-9985-32c8fd205458/9673b332-b1ed-481c-ad2c-77a34f76cbb1"
 					(reference "#PWRENC01")
 					(unit 1)
@@
 		(instances
 			(project "encoder"
-				(path "/23e15ccf-2162-4caa-a05b-71e788486361/627dfe32-6c71-41ac-99ad-61f4ee65e4fe"
+				(path "/dc3b1c6f-161a-46e4-9985-32c8fd205458/9673b332-b1ed-481c-ad2c-77a34f76cbb1"
 					(reference "#PWRENC02")
 					(unit 1)
@@
 		(instances
 			(project "encoder"
-				(path "/23e15ccf-2162-4caa-a05b-71e788486361/627dfe32-6c71-41ac-99ad-61f4ee65e4fe"
+				(path "/dc3b1c6f-161a-46e4-9985-32c8fd205458/9673b332-b1ed-481c-ad2c-77a34f76cbb1"
 					(reference "#PWRENC03")
 					(unit 1)
@@
 		(instances
 			(project "encoder"
-				(path "/23e15ccf-2162-4caa-a05b-71e788486361/627dfe32-6c71-41ac-99ad-61f4ee65e4fe"
+				(path "/dc3b1c6f-161a-46e4-9985-32c8fd205458/9673b332-b1ed-481c-ad2c-77a34f76cbb1"
 					(reference "#PWRENC04")
 					(unit 1)
@@
 		(instances
 			(project "encoder"
-				(path "/23e15ccf-2162-4caa-a05b-71e788486361/627dfe32-6c71-41ac-99ad-61f4ee65e4fe"
+				(path "/dc3b1c6f-161a-46e4-9985-32c8fd205458/9673b332-b1ed-481c-ad2c-77a34f76cbb1"
 					(reference "C40")
 					(unit 1)
@@
 		(instances
 			(project "encoder"
-				(path "/23e15ccf-2162-4caa-a05b-71e788486361/627dfe32-6c71-41ac-99ad-61f4ee65e4fe"
+				(path "/dc3b1c6f-161a-46e4-9985-32c8fd205458/9673b332-b1ed-481c-ad2c-77a34f76cbb1"
 					(reference "#PWRENC05")
 					(unit 1)
@@
 		(instances
 			(project "encoder"
-				(path "/23e15ccf-2162-4caa-a05b-71e788486361/627dfe32-6c71-41ac-99ad-61f4ee65e4fe"
+				(path "/dc3b1c6f-161a-46e4-9985-32c8fd205458/9673b332-b1ed-481c-ad2c-77a34f76cbb1"
 					(reference "#PWRENC06")
 					(unit 1)
@@
 		)
 	)
+	(symbol
+		(lib_id "Device:R")
+		(at 71.12 66.04 0)
+		(unit 1)
+		(exclude_from_sim no)
+		(in_bom yes)
+		(on_board yes)
+		(dnp no)
+		(fields_autoplaced no)
+		(property "Reference" "R24"
+			(at 73.66 64.77 0)
+			(effects
+				(font
+					(size 1.27 1.27)
+				)
+				(justify left)
+			)
+		)
+		(property "Value" "10k 1%"
+			(at 73.66 67.31 0)
+			(effects
+				(font
+					(size 1.27 1.27)
+				)
+				(justify left)
+			)
+		)
+		(property "Footprint" "Resistor_SMD:R_0402_1005Metric"
+			(at 69.342 66.04 90)
+			(effects
+				(font
+					(size 1.27 1.27)
+				)
+				(hide yes)
+			)
+		)
+		(property "LCSC" "C25744"
+			(at 73.66 71.1199 0)
+			(hide yes)
+			(effects
+				(font
+					(size 1.27 1.27)
+				)
+				(justify left)
+			)
+		)
+		(property "MPN" "0402WGF1002TCE"
+			(at 73.66 71.1199 0)
+			(hide yes)
+			(effects
+				(font
+					(size 1.27 1.27)
+				)
+				(justify left)
+			)
+		)
+		(pin "1"
+		)
+		(pin "2"
+		)
+		(instances
+			(project "encoder"
+				(path "/dc3b1c6f-161a-46e4-9985-32c8fd205458/9673b332-b1ed-481c-ad2c-77a34f76cbb1"
+					(reference "R24")
+					(unit 1)
+				)
+			)
+		)
+	)
+	(symbol
+		(lib_id "power:+3V3")
+		(at 71.12 59.69 0)
+		(unit 1)
+		(exclude_from_sim no)
+		(in_bom yes)
+		(on_board yes)
+		(dnp no)
+		(fields_autoplaced no)
+		(property "Reference" "#PWRENC07"
+			(at 71.12 55.88 0.0000)
+			(effects
+				(font
+					(size 1.27 1.27)
+				)
+				(justify left)
+				(hide yes)
+			)
+		)
+		(property "Value" "+3V3"
+			(at 71.12 54.61 0)
+			(effects
+				(font
+					(size 1.27 1.27)
+				)
+			)
+		)
+		(pin "1"
+		)
+		(instances
+			(project "encoder"
+				(path "/dc3b1c6f-161a-46e4-9985-32c8fd205458/9673b332-b1ed-481c-ad2c-77a34f76cbb1"
+					(reference "#PWRENC07")
+					(unit 1)
+				)
+			)
+		)
+	)
 	(wire
 		(pts
@@
 		(pts
 			(xy 96.52 69.85) (xy 96.52 72.39)
+		)
+		(stroke
+			(width 0)
+			(type default)
+		)
+	)
+	(wire
+		(pts
+			(xy 71.12 62.23) (xy 71.12 59.69)
+		)
+		(stroke
+			(width 0)
+			(type default)
+		)
+	)
+	(wire
+		(pts
+			(xy 71.12 69.85) (xy 71.12 72.39)
 		)
 		(stroke
@@
 		)
 	)
+	(hierarchical_label "ENC_CS"
+		(shape input)
+		(at 71.12 72.39 270)
+		(effects
+			(font
+				(size 1.27 1.27)
+			)
+			(justify right)
+		)
+	)
 	(no_connect
 		(at 152.4 91.44)
@@
 		(at 152.4 93.98)
 	)
-	(text "AS5047P 3.3 V operation: VDD and VDD3V3 tied to 3.3 V, one 100 nF (DS000324 Fig. 10).\nTEST (pin 5) to GND per pin table. ABI / UVW / PWM outputs unused.\nSPI mode 1, up to 10 MHz, on its own SPI port (SPI3).\nPlace alone on the motor-facing side at the board center. Magnet 6 x 2.5 mm diametric,\ngap 1 to 2 mm. Keep phase and pass-through currents >= 12 mm away."
+	(text "AS5047P 3.3 V operation: VDD and VDD3V3 tied to 3.3 V, one 100 nF (DS000324 Fig. 10).\nTEST (pin 5) to GND per pin table. ABI / UVW / PWM outputs unused.\nR24 holds CSn high while the MCU is in reset or ROM DFU (inputs must not float, DS p.4).\nSPI mode 1, up to 10 MHz, on its own SPI port (SPI3).\nPlace alone on the motor-facing side at the board center. Magnet 6 x 2.5 mm diametric,\ngap 1 to 2 mm. Keep phase and pass-through currents >= 12 mm away."
 		(exclude_from_sim no)
 		(at 25.4 137.16 0.0000)

Commit message: Route the 6-layer board and finalize parts for ordering
The 45 x 45 mm board is fully routed on six layers (F / GND / SIG /
SIG / PWR / B, 2 oz outer, 1 oz inner): DRC 0 errors, 0 unconnected,
schematic parity 0. Four layers could not route the DRV-to-MCU links
without moving the power or input stage.

- Encoder shares the DRV8353's SPI3 bus, as on the PoC; PA5-PA7 are
  unused. R25 pulls DRV nSCS up, since the DRV's logic inputs have an
  internal pull-down. The SDO / MISO pin-type warning is an ERC
  exclusion with a note.
- MCU is now the STM32G473CEU6: the G474 without the unused HRTIM,
  checked pin for pin against both datasheets, in stock and cheaper.
- Male XT30PW-M power connectors, HCS1206 shunts, SWD pads at the
  board edge.
- Design doc and review notes updated for the new stack-up, shared
  bus and MCU.

Co-Authored-By: Claude Opus 5.5 <noreply@anthropic.com>
Connections:
- net ENC_MISO renamed DRV_SDO
- net ENC_MOSI renamed DRV_SDI
- net ENC_SCK renamed DRV_SCLK
Other:
- note added: "AS5047P 3.3 V operation: VDD and VDD3V3 tied to 3.3 V, one 100 nF (DS000324 Fig. 10). TEST (pin 5) to GND per pin table. ABI / UVW / PWM outputs unused. R24 holds CSn high while the MCU is in reset or ROM DFU (inputs must not float, DS p.4). SPI mode 1, up to 10 MHz, on its own SPI port (SPI1). Place alone on the motor-facing side at the board center. Magnet 6 x 2.5 mm diametric, gap 1 to 2 mm. K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"
- note removed: "AS5047P 3.3 V operation: VDD and VDD3V3 tied to 3.3 V, one 100 nF (DS000324 Fig. 10). TEST (pin 5) to GND per pin table. ABI / UVW / PWM outputs unused. R24 holds CSn high while the MCU is in reset or ROM DFU (inputs must not float, DS p.4). SPI mode 1, up to 10 MHz, on its own SPI port (SPI3). Place alone on the motor-facing side at the board center. Magnet 6 x 2.5 mm diametric, gap 1 to 2 mm. K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"
Changed lines of the file:
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@@
 		(comment 2 "specs/pmsm-controller/design-electronics.md")
 	)
-	(text "AS5047P 3.3 V operation: VDD and VDD3V3 tied to 3.3 V, one 100 nF (DS000324 Fig. 10).\nTEST (pin 5) to GND per pin table. ABI / UVW / PWM outputs unused.\nR24 holds CSn high while the MCU is in reset or ROM DFU (inputs must not float, DS p.4).\nSPI mode 1, up to 10 MHz, on its own SPI port (SPI3).\nPlace alone on the motor-facing side at the board center. Magnet 6 x 2.5 mm diametric,\ngap 1 to 2 mm. Keep phase and pass-through currents >= 12 mm away."
+	(text "AS5047P 3.3 V operation: VDD and VDD3V3 tied to 3.3 V, one 100 nF (DS000324 Fig. 10).\nTEST (pin 5) to GND per pin table. ABI / UVW / PWM outputs unused.\nR24 holds CSn high while the MCU is in reset or ROM DFU (inputs must not float, DS p.4).\nSPI mode 1, up to 10 MHz, on its own SPI port (SPI1).\nPlace alone on the motor-facing side at the board center. Magnet 6 x 2.5 mm diametric,\ngap 1 to 2 mm. Keep phase and pass-through currents >= 12 mm away."
 		(exclude_from_sim no)
 		(at 25.4 137.16 0)
@@
 		)
 	)
-	(hierarchical_label "ENC_SCK"
+	(hierarchical_label "DRV_SCLK"
 		(shape input)
 		(at 119.38 93.98 180)
@@
 		)
 	)
-	(hierarchical_label "ENC_MOSI"
+	(hierarchical_label "DRV_SDI"
 		(shape input)
 		(at 119.38 88.9 180)
@@
 		)
 	)
-	(hierarchical_label "ENC_MISO"
+	(hierarchical_label "DRV_SDO"
 		(shape output)
 		(at 119.38 91.44 180)
